File: GS_LPC_RadioBoard.kicad_sch (KiCad schematic)
At the start: 19 parts, among them J1 142-0701-886, J3 Conn_01x04_Pin, J4 Conn_01x07_Pin, Y1 NX2016SA-26M-STD-CZS-1

Commit message: finish first wiring
Parts:
- removed J1: 142-0701-886, footprints:TAOGLAS_EMPCB.SMAFSTJ.B.HT, symbol 142-0701-886:142-0701-886
- removed J3: Conn_01x04_Pin, Connector_PinHeader_2.00mm:PinHeader_1x04_P2.00mm_Vertical, symbol Connector:Conn_01x04_Pin
- added J2: Conn_01x05_Pin, Connector_PinHeader_2.00mm:PinHeader_1x05_P2.00mm_Vertical, symbol Connector:Conn_01x05_Pin
- added J3: EMPCB.SMAFSTJ.B.HT, EMPCB.SMAFSTJ.B.HT:TAOGLAS_EMPCB.SMAFSTJ.B.HT, symbol EMPCB.SMAFSTJ.B.HT:EMPCB.SMAFSTJ.B.HT
Connections:
- net BUSY: now also J2.2 (Pin_2)
- net DIO1: now also J2.3 (Pin_3)
- net DIO2: now also J2.4 (Pin_4)
- net DIO3: now also J2.5 (Pin_5)
- net GND: now also J2.1 (Pin_1), J3.SH1; no longer J4.7 (Pin_7)
- net VDD_RADIO: now also J4.7 (Pin_7)
- net at C4.2: now also J3.1

Commit message: version with minor adjustement
Parts:
- J3: footprint EMPCB.SMAFSTJ.B.HT:TAOGLAS_EMPCB.SMAFSTJ.B.HT -> footprints:TAOGLAS_EMPCB.SMAFSTJ.B.HT
- renumbered J4 to J1
Changed lines of the file:
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@@
       (effects (font (size 1.27 1.27)) (justify left))
     )
-    (property "Footprint" "EMPCB.SMAFSTJ.B.HT:TAOGLAS_EMPCB.SMAFSTJ.B.HT" (at 220.98 36.83 0)
+    (property "Footprint" "footprints:TAOGLAS_EMPCB.SMAFSTJ.B.HT" (at 220.98 36.83 0)
       (effects (font (size 1.27 1.27)) (justify bottom) hide)
     )
@@
   (symbol (lib_id "Connector:Conn_01x07_Pin") (at 168.91 111.76 0) (unit 1)
     (in_bom yes) (on_board yes) (dnp no) (fields_autoplaced)
-    (property "Reference" "J4" (at 169.545 99.06 0)
+    (property "Reference" "J1" (at 169.545 99.06 0)
       (effects (font (size 1.27 1.27)))
     )
@@
       (project "GS_LPC_RadioBoard"
         (path "/0c275095-00c0-41ae-b08c-e5453f1b3f88"
-          (reference "J4") (unit 1)
+          (reference "J1") (unit 1)
         )
       )
